File: simple-amplifier/simple-amplifier.kicad_sch (KiCad schematic)
At the start: 8 parts, among them Q1 BC559

Commit message: Small changes
Parts:
- C3: value C_Polarized -> 100pf
Changed lines of the file:
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@@
 			)
 		)
-		(property "Value" "C_Polarized"
+		(property "Value" "100pf"
 			(at 97.409 77.47 90)
 			(effects
